File: line_electrodes/line_electrodes.kicad_pcb (KiCad board)
At the start: 2 copper layers, 27 x 43 mm, 2 parts, among them J1 Line electrodes, J2 SM12B-GHS

Commit message: wip
Routing:
- net Net-(J1-Pin_12): track 0.00 -> 30.9 mm
- net Net-(J1-Pin_11): track 0.00 -> 30.5 mm
- net Net-(J1-Pin_10): track 0.00 -> 30.2 mm
- net Net-(J1-Pin_9): track 0.00 -> 29.9 mm
- net Net-(J1-Pin_4): track 0.00 -> 29.9 mm
- net Net-(J1-Pin_8): track 0.00 -> 29.6 mm
- net Net-(J1-Pin_5): track 0.00 -> 29.6 mm
- net Net-(J1-Pin_7): track 0.00 -> 29.3 mm
- net Net-(J1-Pin_6): track 0.00 -> 29.3 mm
Changed lines of the file:
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@@
 	)
 	(segment
-		(start 17 34)
-		(end 20.375 37.375)
+		(start 29.125 34.875)
+		(end 31 33)
+		(width 0.5)
+		(layer "F.Cu")
+		(net "Net-(J1-Pin_9)")
+	)
+	(segment
+		(start 29.125 49.15)
+		(end 29.125 34.875)
+		(width 0.5)
+		(layer "F.Cu")
+		(net "Net-(J1-Pin_9)")
+	)
+	(segment
+		(start 31 33)
+		(end 31 20)
+		(width 0.5)
+		(layer "F.Cu")
+		(net "Net-(J1-Pin_9)")
+	)
+	(segment
+		(start 33 20)
+		(end 33 33)
+		(width 0.5)
+		(layer "F.Cu")
+		(net "Net-(J1-Pin_10)")
+	)
+	(segment
+		(start 30.375 35.625)
+		(end 30.375 49.15)
+		(width 0.5)
+		(layer "F.Cu")
+		(net "Net-(J1-Pin_10)")
+	)
+	(segment
+		(start 33 33)
+		(end 30.375 35.625)
+		(width 0.5)
+		(layer "F.Cu")
+		(net "Net-(J1-Pin_10)")
+	)
+	(segment
+		(start 17 20)
+		(end 17 33)
 		(width 0.5)
 		(layer "F.Cu")
@@
 	)
 	(segment
-		(start 17 20)
-		(end 17 34)
+		(start 17 33)
+		(end 20.375 36.375)
 		(width 0.5)
 		(layer "F.Cu")
@@
 	)
 	(segment
-		(start 20.375 37.375)
+		(start 20.375 36.375)
 		(end 20.375 49.15)
 		(width 0.5)
@@
 	)
 	(segment
-		(start 19 34)
-		(end 21.625 36.625)
+		(start 27 32.75)
+		(end 27 20)
+		(width 0.5)
+		(layer "F.Cu")
+		(net "Net-(J1-Pin_7)")
+	)
+	(segment
+		(start 26.625 49.15)
+		(end 26.625 33.125)
+		(width 0.5)
+		(layer "F.Cu")
+		(net "Net-(J1-Pin_7)")
+	)
+	(segment
+		(start 26.625 33.125)
+		(end 27 32.75)
+		(width 0.5)
+		(layer "F.Cu")
+		(net "Net-(J1-Pin_7)")
+	)
+	(segment
+		(start 29 20)
+		(end 29 33)
+		(width 0.5)
+		(layer "F.Cu")
+		(net "Net-(J1-Pin_8)")
+	)
+	(segment
+		(start 29 33)
+		(end 27.875 34.125)
+		(width 0.5)
+		(layer "F.Cu")
+		(net "Net-(J1-Pin_8)")
+	)
+	(segment
+		(start 27.875 34.125)
+		(end 27.875 49.15)
+		(width 0.5)
+		(layer "F.Cu")
+		(net "Net-(J1-Pin_8)")
+	)
+	(segment
+		(start 35 20)
+		(end 35 33)
+		(width 0.5)
+		(layer "F.Cu")
+		(net "Net-(J1-Pin_11)")
+	)
+	(segment
+		(start 35 33)
+		(end 31.625 36.375)
+		(width 0.5)
+		(layer "F.Cu")
+		(net "Net-(J1-Pin_11)")
+	)
+	(segment
+		(start 31.625 36.375)
+		(end 31.625 49.15)
+		(width 0.5)
+		(layer "F.Cu")
+		(net "Net-(J1-Pin_11)")
+	)
+	(segment
+		(start 19 33)
+		(end 21.625 35.625)
 		(width 0.5)
 		(layer "F.Cu")
@@
 	)
 	(segment
-		(start 21.625 36.625)
+		(start 19 20)
+		(end 19 33)
+		(width 0.5)
+		(layer "F.Cu")
+		(net "Net-(J1-Pin_3)")
+	)
+	(segment
+		(start 21.625 35.625)
 		(end 21.625 49.15)
 		(width 0.5)
@@
 	)
 	(segment
-		(start 19 20)
-		(end 19 34)
-		(width 0.5)
-		(layer "F.Cu")
-		(net "Net-(J1-Pin_3)")
-	)
-	(segment
-		(start 19.125 40.125)
+		(start 37 33)
+		(end 32.875 37.125)
+		(width 0.5)
+		(layer "F.Cu")
+		(net "Net-(J1-Pin_12)")
+	)
+	(segment
+		(start 37 20)
+		(end 37 33)
+		(width 0.5)
+		(layer "F.Cu")
+		(net "Net-(J1-Pin_12)")
+	)
+	(segment
+		(start 32.875 37.125)
+		(end 32.875 49.15)
+		(width 0.5)
+		(layer "F.Cu")
+		(net "Net-(J1-Pin_12)")
+	)
+	(segment
+		(start 22.875 34.875)
+		(end 22.875 49.15)
+		(width 0.5)
+		(layer "F.Cu")
+		(net "Net-(J1-Pin_4)")
+	)
+	(segment
+		(start 21 33)
+		(end 22.875 34.875)
+		(width 0.5)
+		(layer "F.Cu")
+		(net "Net-(J1-Pin_4)")
+	)
+	(segment
+		(start 21 20)
+		(end 21 33)
+		(width 0.5)
+		(layer "F.Cu")
+		(net "Net-(J1-Pin_4)")
+	)
+	(segment
+		(start 23 33)
+		(end 24.125 34.125)
+		(width 0.5)
+		(layer "F.Cu")
+		(net "Net-(J1-Pin_5)")
+	)
+	(segment
+		(start 23 20)
+		(end 23 33)
+		(width 0.5)
+		(layer "F.Cu")
+		(net "Net-(J1-Pin_5)")
+	)
+	(segment
+		(start 24.125 34.125)
+		(end 24.125 49.15)
+		(width 0.5)
+		(layer "F.Cu")
+		(net "Net-(J1-Pin_5)")
+	)
+	(segment
+		(start 25.375 33.125)
+		(end 25 32.75)
+		(width 0.5)
+		(layer "F.Cu")
+		(net "Net-(J1-Pin_6)")
+	)
+	(segment
+		(start 25.375 49.15)
+		(end 25.375 33.125)
+		(width 0.5)
+		(layer "F.Cu")
+		(net "Net-(J1-Pin_6)")
+	)
+	(segment
+		(start 25 20)
+		(end 25 32.75)
+		(width 0.5)
+		(layer "F.Cu")
+		(net "Net-(J1-Pin_6)")
+	)
+	(segment
+		(start 15 20)
+		(end 15 33.5)
+		(width 0.5)
+		(layer "F.Cu")
+		(net "Net-(J1-Pin_1)")
+	)
+	(segment
+		(start 15 33.5)
+		(end 19.125 37.625)
+		(width 0.5)
+		(layer "F.Cu")
+		(net "Net-(J1-Pin_1)")
+	)
+	(segment
+		(start 19.125 37.625)
 		(end 19.125 49.15)
 		(width 0.5)
 		(layer "F.Cu")
-		(net "Net-(J1-Pin_1)")
-	)
-	(segment
-		(start 15 20)
-		(end 15 36)
-		(width 0.5)
-		(layer "F.Cu")
-		(net "Net-(J1-Pin_1)")
-	)
-	(segment
-		(start 15 36)
-		(end 19.125 40.125)
-		(width 0.5)
-		(layer "F.Cu")
